File: TAD5142_Module.kicad_pcb (KiCad board)
At the start: 4 copper layers, 40 x 27 mm, 20 parts, among them J1 Conn_01x02, J2 AudioJack2_Ground, J3 Conn_01x05, U1 AP7361EA-33E-13, U2 TAD5142IRGER

Commit message: Add PCB dimensions.
Other:
- board text added: "UNIT: mm t: 1.6"
